File: bmw.sch (EAGLE design)
At the start: 64 parts, among them U1 LPC1114FDH28, U2 S25FL208K, U3 MCP23008, U4 MCP1252

Commit message: revision 2
Parts:
- removed PWR_LED: (no value), led:LEDCHIPLED_1206
- removed SW_BL: (no value), ivan:DS01
- removed SW_D: 219-02, switch-dil:219-02
- added C13, C14: 0.1uF, rcl:C-EUC0805
- added C15, C16: 4.7uF, rcl:C-EUC0805
- added CHG, PWR: (no value), led:LEDCHIPLED_0805
- added CON_USB: CON-USB-F-MINI-B, dp_devices:CON-USB-F-MINI-B
- added JP_BL: (no value), pinhead:PINHD-1X2
- added PCB1: PCB_DP_RECTANGLE-43X70, dp_devices:PCB_DP_RECTANGLE-43X70
- added R26: (no value), rcl:R-US_R0805
- added R27: 10K, rcl:R-US_R0805
- added SW_DIP: 219-02, switch-dil:219-02
- added U5: MCP73831/2, ivan:MCP73831/2
- C1, C10, C11, C2, C3, C4, C5, C6: device rcl:C-EUC0603 -> rcl:C-EUC0805
- C12: device rcl:C-EUC1206 -> rcl:C-EUC0805
- LED1, LED2, LED3, LED4: device led:LEDCHIPLED_1206 -> led:LEDCHIPLED_0805
- R1, R10, R11, R12, R13, R14, R15, R16, R17, R18, R19, R7: device rcl:R-US_R0603 -> rcl:R-US_R0805
- R20, R22, R24: value 0 -> DNP; device rcl:R-US_R0402 -> rcl:R-US_R0603
- R21, R23, R25: device rcl:R-US_R0402 -> rcl:R-US_R0603
- R8, R9: value 1K -> 10K; device rcl:R-US_R0603 -> rcl:R-US_R0805
- renumbered S3 to SW_B0, S4 to SW_B1
Connections:
- new net N$15: CHG.C, R26.2
- new net N$16: R26.1, U5.STAT
- new net N$17: R27.2, U5.PROG
- net +3V3: now also PWR.A; no longer PWR_LED.A
- net BL: now also JP_BL.2; no longer SW_BL.2
- net GND: now also C13.2, C14.2, C15.1, C16.1, CON_USBUSB.GND, JP_BL.1, R27.1, SW_DIP.1, SW_DIP.2, U5.VSS; no longer SW_BL.1, SW_D.1, SW_D.2
- net I2C_SCL: now also JP_I2C.1; no longer JP_I2C.2
- net I2C_SDA: now also JP_I2C.2; no longer JP_I2C.1
- net LIPO_3.7V: now also C16.2, U5.VBAT
- net N$1: now also SW_DIP.4; no longer SW_D.4
- net N$14: now also SW_DIP.3; no longer SW_D.3
- net N$4: now also PWR.C; no longer PWR_LED.C
- net SW_D0: now also C13.1
- net SW_D1: now also C14.1
- net USB_5V: now also C15.2, CHG.A, CON_USBUSB.VUSB, U5.VDD; no longer JP_UART.3
Other:
- note added: "3.3V / 120mA Switch Capacitor Regulator"
- note added: "ARM Bare Metal Widget Rev. 2"
- note added: "Bootloader Jumper"
- note added: "CC-BY-4.0"
- note added: "JST LiPo Connector for Battery Power"
- note added: "LiPo Charger"
- note added: "Limit charging current to 1000V/10K = 100mA for now"
- note added: "PCB and Mounting Holes"
- note added: "USB Mini-B Connector for USB Power"
- note added: "USB/LiPo/Off Power Switch"
- note added: "http://theanine.io"
- note removed: "120mA @ 3.3V Switch Capacitor Regulator"
- note removed: "ARM Bare Metal Widget Rev. 1.0"
- note removed: "Bootloader Switch"
- note removed: "USB/LiPo/Off Power Selector Switch"
- note removed: "http://vsdev.me"
- moved on the sheet: C12, C3, C4, C7, C8, C9, CON_BAT, JP_UART, R1, R10, R11, R16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

Commit message: fix spi flash value in schematic
Parts:
- U2: value S25FL208K -> S25FL216K
Changed lines of the file:
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@@
 <parts>
 <part name="U1" library="ivan" deviceset="LPC1114FDH28" device=""/>
-<part name="U2" library="ivan" deviceset="S25FL208K" device=""/>
+<part name="U2" library="ivan" deviceset="S25FL208K" device="" value="S25FL216K"/>
 <part name="+3V1" library="supply1" deviceset="+3V3" device=""/>
 <part name="GND1" library="supply1" deviceset="GND" device=""/>
